Commit message: Set initial position in sim using yaml by updating xacro, update moveit_configs_builder.

File: src/lbr_fri_ros2_stack/lbr_description/urdf/med7/med7.urdf.xacro (robot description, xacro)
@@ -7,4 +7,5 @@
     <xacro:arg name="port_id" default="30200" />
     <xacro:arg name="sim" default="true" />
+    <xacro:arg name="initial_positions_file" default="initial_positions.yaml" />
     <!-- fixed to world, see http://classic.gazebosim.org/tutorials?tut=ros_urdf&cat=connect_ros -->
     <link name="world" />
@@ -20,4 +21,4 @@
     </joint>
     <!-- med -->
-    <xacro:med7 robot_name="$(arg robot_name)" port_id="$(arg port_id)" sim="$(arg sim)" />
+    <xacro:med7 robot_name="$(arg robot_name)" port_id="$(arg port_id)" sim="$(arg sim)" initial_positions_file="$(arg initial_positions_file)"/>
 </robot>

File: src/lbr_fri_ros2_stack/lbr_description/urdf/med7/med7_description.urdf.xacro (robot description, xacro)
@@ -25,5 +25,5 @@
     <!-- robot as extracted via https://github.com/syuntoku14/fusion2urdf -->
     <xacro:macro name="med7"
-        params="robot_name:=^|lbr port_id:=^|30200 sim:=^|true">
+        params="robot_name:=^|lbr port_id:=^|30200 sim:=^|true initial_positions_file:=^|initial_positions.yaml">
         <link name="plank">
             <inertial>
@@ -364,5 +364,6 @@
             A7_velocity_limit="${A7_velocity_limit * PI / 180}"
             max_torque="${effort_limit}"
-            sim="${sim}" remote_host="INADDR_ANY" port_id="${port_id}" />
+            sim="${sim}" remote_host="INADDR_ANY" port_id="${port_id}"
+            initial_positions_file="${initial_positions_file}"/>
     </xacro:macro>
 </robot>

File: src/lbr_fri_ros2_stack/lbr_ros2_control/config/lbr_system_interface.xacro (robot description, xacro)
@@ -3,4 +3,5 @@
     <xacro:macro name="lbr_system_interface"
         params="
+        initial_positions_file
         A1_position_limit
         A2_position_limit
@@ -106,5 +107,5 @@
             <!-- define joints and command/state interfaces for each joint -->
             <xacro:macro name="joint_interface"
-                params="name min_position max_position max_velocity max_torque sim">
+                params="name min_position max_position max_velocity max_torque sim default_position">
                 <joint name="${name}">
                     <param name="min_position">${min_position}</param>
@@ -120,5 +121,9 @@
                         <param name="max"> ${max_torque}</param>
                     </command_interface>
-                    <state_interface name="position" />
+                    <state_interface name="position">
+                        <xacro:if value="${sim}">
+                            <param name="initial_value">${default_position}</param>
+                        </xacro:if>
+                    </state_interface>
                     <state_interface name="velocity" />
                     <state_interface name="effort" />
@@ -131,25 +136,26 @@
                 </joint>
             </xacro:macro>
+            <xacro:property name="initial_positions" value="${xacro.load_yaml(initial_positions_file)['initial_positions']}"/>
             <xacro:joint_interface name="A1" min_position="-${A1_position_limit}"
                 max_position="${A1_position_limit}" max_velocity="${A1_velocity_limit}"
-                max_torque="${max_torque}" sim="${sim}" />
+                max_torque="${max_torque}" sim="${sim}" default_position="${initial_positions['A1']}"/>
             <xacro:joint_interface name="A2" min_position="-${A2_position_limit}"
                 max_position="${A2_position_limit}" max_velocity="${A2_velocity_limit}"
-                max_torque="${max_torque}" sim="${sim}" />
+                max_torque="${max_torque}" sim="${sim}" default_position="${initial_positions['A2']}"/>
             <xacro:joint_interface name="A3" min_position="-${A3_position_limit}"
                 max_position="${A3_position_limit}" max_velocity="${A3_velocity_limit}"
-                max_torque="${max_torque}" sim="${sim}" />
+                max_torque="${max_torque}" sim="${sim}" default_position="${initial_positions['A3']}"/>
             <xacro:joint_interface name="A4" min_position="-${A4_position_limit}"
                 max_position="${A4_position_limit}" max_velocity="${A4_velocity_limit}"
-                max_torque="${max_torque}" sim="${sim}" />
+                max_torque="${max_torque}" sim="${sim}" default_position="${initial_positions['A4']}"/>
             <xacro:joint_interface name="A5" min_position="-${A5_position_limit}"
                 max_position="${A5_position_limit}" max_velocity="${A5_velocity_limit}"
-                max_torque="${max_torque}" sim="${sim}" />
+                max_torque="${max_torque}" sim="${sim}" default_position="${initial_positions['A5']}"/>
             <xacro:joint_interface name="A6" min_position="-${A6_position_limit}"
                 max_position="${A6_position_limit}" max_velocity="${A6_velocity_limit}"
-                max_torque="${max_torque}" sim="${sim}" />
+                max_torque="${max_torque}" sim="${sim}" default_position="${initial_positions['A6']}"/>
             <xacro:joint_interface name="A7" min_position="-${A7_position_limit}"
                 max_position="${A7_position_limit}" max_velocity="${A7_velocity_limit}"
-                max_torque="${max_torque}" sim="${sim}" />
+                max_torque="${max_torque}" sim="${sim}" default_position="${initial_positions['A7']}"/>
         </ros2_control>
     </xacro:macro>
