Commit message: Remove plank link.

File: src/lbr_fri_ros2_stack/lbr_description/gazebo/lbr_gazebo.xacro (robot description, xacro)
@@ -44,6 +44,4 @@
         <xacro:gazebo_joint_reference name="joint_tool" />
         <xacro:gazebo_link_reference name="link_tool" />
-        <xacro:gazebo_joint_reference name="world_plank_joint" />
-        <xacro:gazebo_link_reference name="plank" />
     </xacro:macro>
 </robot>

File: src/lbr_fri_ros2_stack/lbr_description/urdf/med7/med7.urdf.xacro (robot description, xacro)
@@ -16,8 +16,4 @@
         <child link="link_0" />
     </joint>
-    <joint name="world_plank_joint" type="fixed">
-        <parent link="world" />
-        <child link="plank" />
-    </joint>
     <!-- med -->
     <xacro:med7 robot_name="$(arg robot_name)" port_id="$(arg port_id)" sim="$(arg sim)" initial_positions_file="$(arg initial_positions_file)"/>

File: src/lbr_fri_ros2_stack/lbr_description/urdf/med7/med7_description.urdf.xacro (robot description, xacro)
@@ -26,28 +26,4 @@
     <xacro:macro name="med7"
         params="robot_name:=^|lbr port_id:=^|30200 sim:=^|true initial_positions_file:=^|initial_positions.yaml">
-        <link name="plank">
-            <inertial>
-                <origin rpy="0 0 0" xyz="-0.001896 0.0 0.076263" />
-                <mass value="7.143112" />
-                <inertia ixx="0.038694" ixy="0.0" ixz="-0.000686" iyy="0.039461" iyz="0.0"
-                    izz="0.054387" />
-            </inertial>
-            <visual>
-                <origin rpy="0 0 0" xyz="-0.47 0 -0.017" />
-                <geometry>
-                    <box size="0.64 1.1 0.02"/>
-                </geometry>
-                <material name="gray">
-                    <color rgba="0.5 0.5 0.5 1.0" />
-                </material>
-            </visual>
-            <!-- maybe need to turn this on, for now it is off for spawning in gazebo -->
-            <!-- <collision>
-                <origin rpy="0 0 0" xyz="-0.47 0 -0.017" />
-                <geometry>
-                    <box size="0.64 1.1 0.02"/>
-                </geometry>
-            </collision> -->
-        </link>
         <link name="link_0">
             <inertial>
